Commit message: save1

File: src/mbot_description/urdf/xacro/gazebo/mbot_base_gazebo.xacro (robot description, xacro)
@@ -3,5 +3,5 @@
     <!-- PROPERTY LIST -->
     <xacro:property name="M_PI" value="3.1415926"/>
-    <xacro:property name="base_mass"   value="19.67835472" />
+    <xacro:property name="base_mass"   value="19.44064455" />
     <xacro:property name="wheel_mass"   value="0.478515278465427" />
     <xacro:property name="caster_mass"   value="0.205283816888508" />
@@ -25,10 +25,10 @@
             <mass value="${m}" />
             <inertia
-              ixx="3.39695676"
-              ixy="-0.00097485"
-              ixz="0.35282533"
-              iyy="3.41361621"
-              iyz="-0.00013272"
-              izz="1.02770643" />
+              ixx="3.40354705"
+              ixy="-0.00036197"
+              ixz="0.332666732"
+              iyy="3.40038142"
+              iyz="0.00198404"
+              izz="1.03448983" />
           </inertial>
     </xacro:macro>

File: src/mbot_description/urdf/xacro/sensors/lidar_gazebo.xacro (robot description, xacro)
@@ -43,5 +43,5 @@
             <sensor type="ray" name="rplidar">
                 <pose>0 0 0 0 0 0</pose>
-                <visualize>true</visualize>
+                <visualize>false</visualize>
                 <update_rate>5.5</update_rate>
                 <ray>
@@ -55,5 +55,5 @@
                     </scan>
                     <range>
-                      <min>0.10</min>
+                      <min>0.5</min>
                       <max>20</max>
                       <resolution>0.01</resolution>
